File: rev_1/Beerduino.kicad_pcb (KiCad board)
At the start: 2 copper layers, 68 x 53 mm, 54 parts, among them J1 ICSP, J2 Header1, J3 Header2, J4 PWR, J5 Analog, J6 RAW, J7 Reg_jump, J8 USB_B_Micro, U1 ATmega168P-20A, U3 LE33CZ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

Commit message: rev1 initial
Parts:
- removed DS1: BC56-12GWA, Display:DIPS1524W50P254L3760H810Q12N
- added DS2: BC56-12GWA, Display:3digit, F.Cu at (106.7, 89.2)

Commit message: documentation
Parts:
- removed G***: LOGO, LOGO
Connections:
- U4 pad 18: unconnected-(U4-GND-Pad18) -> GND
- U4 pad 25: unconnected-(U4-GND-Pad25) -> GND
- U4 pad 34: unconnected-(U4-GND-Pad34) -> GND
- U4 pad 45: unconnected-(U4-AGND-Pad45) -> GND
- U4 pad 9: unconnected-(U4-GND-Pad9) -> GND
Routing:
- net GND: track 28.2 -> 44.6 mm
