File: rev_1/Beerduino.kicad_sch (KiCad schematic)
At the start: 39 parts, among them J1 ICSP, J2 Header1, J3 Header2, J4 PWR, J5 Analog, J6 RAW, J7 Reg_jump, U1 ATmega168P-20A, U3 LE33CZ, U5 L78L05_SOT89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

Commit message: rev1 initial
Parts:
- removed DS1: BC56-12GWA, Display:DIPS1524W50P254L3760H810Q12N, symbol BC56-12GWA:BC56-12GWA
- added DS2: BC56-12GWA, symbol display:3_digit_no_dots
Connections:
- net D11: now also DS2.8 (1)
- net D12: now also DS2.9 (2)
- net D13: now also DS2.12 (3)
- net at R16.2: now also DS2.10 (f)
- net at R13.2: now also DS2.2 (d)
- net at R14.2: now also DS2.1 (e)
- net at R17.2: now also DS2.11 (a)
- net at R12.2: now also DS2.4 (c)
- net at R11.2: now also DS2.5 (g)
- net at R15.2: now also DS2.7 (b)
Other:
- moved on the sheet: R11, R12, R13, R14, R15, R16, R17

Commit message: documentation
Parts:
- DS2: footprint (none) -> Display:3digit
- J7: value Reg_jump -> LP jumper
Other:
- note added: "3v3 regulator"
- note added: "5v regulator"
- note added: "7-segment display"
- note added: "Aux power"
- note added: "Bottle detector"
- note added: "D2 pulled to ground when in contact with a bottle"
- note added: "ICSP"
- note added: "Input connectors"
- note added: "Microprocessor"
- note added: "Pin 3, 6 removed from footprint"
- note added: "Processor VCC"
- note added: "Uart header"
- note added: "Uno pinheaders"
- note removed: "Vi skal bruge en knap der bliver hamret til stel og så vågner han far sleep og øger en tæller"
- title: (none) -> Beerduino
- moved on the sheet: C1, C10, C17, C2, C3, C4, C6, C7, C8, C9, D1, D2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
